Commit message: Minor optimizing changes

File: map_simu/models/drone_links/drone_links.urdf (robot description, URDF)
Before this commit: robot drone_links, 5 links, 4 joints
Links:
- removed link gps_link
- removed link imu_link
- added link camera_rgb_optical_frame
Joints:
- removed joint camera_joint
- removed joint gps_joint
- removed joint imu_joint
- added joint camera_depth_optical_frame_joint: type fixed, parent camera_rgb_optical_frame, child camera_depth_optical_frame, origin xyz=0 0 0 rpy=0 0 0
- added joint camera_rgb_optical_frame_joint: type fixed, parent base_link, child camera_rgb_optical_frame, origin xyz=0.03 0 0.13 rpy=-2.17079632679 0 -1.57079632679

Commit message: Minor bug fixes

File: map_simu/models/drone_links/drone_links.urdf (robot description, URDF)
Before this commit: robot drone_links, 4 links, 3 joints
Links:
- removed link camera_link
- added link camera_depth_optical_frame

Commit message: Links modified

File: map_simu/models/drone_links/drone_links.urdf (robot description, URDF)
Before this commit: robot drone_links, 4 links, 3 joints
Links:
- added link camera_link
Joints:
- added joint camera_joint: type fixed, parent base_link, child camera_link, origin xyz=0.03 0 0.13 rpy=-1.67079632679 0 -1.57079632679
- joint base_joint: child base_link -> fcu; parent fcu -> base_link
- joint camera_depth_optical_frame_joint: parent camera_rgb_optical_frame -> camera_link
- joint camera_rgb_optical_frame_joint: origin xyz=0.03 0 0.13 rpy=-2.17079632679 0 -1.57079632679 -> xyz=0 0 0 rpy=0 0 0; parent base_link -> camera_link

Commit message: UAV shaking fixed, new Gazebo  model

File: map_simu/models/drone_links/drone_links.urdf (robot description, URDF)
Before this commit: robot drone_links, 5 links, 4 joints
Joints:
- joint camera_joint: origin xyz=0.03 0 0.13 rpy=-1.67079632679 0 -1.57079632679 -> xyz=0.03 0 0.13 rpy=-2.17079632679 0 -1.57079632679
